File: light_blink.kicad_pcb (KiCad board)
At the start: 2 copper layers, 16.5 x 32.5 mm, 14 parts, among them J1 CONN PLUG USB2.0 TYPEA 4POS R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, U1 MCP1702T-3302E/CB, U3 MCP6022T-I/ST

Commit message: Add files via upload
Other:
- board size 16.5 x 32.5 mm -> 16.5 x 19.8 mm
Changed lines of the file:
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@@
 	)
 	(gr_rect
-		(start 69.85 32.258)
+		(start 69.85 45)
 		(end 86.36 64.77)
 		(stroke

Commit message: Add files via upload
Parts:
- added C2: .1UF, Capacitor_SMD:C_0603_1608Metric, F.Cu at (83.2, 53.5)
- moved R8 1.80 mm to (83.5, 60.3)
- moved R9 1.80 mm to (83.5, 56.8)
Routing:
- net GND: track 13.1 -> 21.0 mm, vias 2 -> 3
- net Net-(U1-VOUT): track 19.8 -> 22.8 mm
- net Net-(R7-Pad1): track 3.23 -> 1.59 mm
- net Net-(U3-VOUTB): track 10.9 -> 10.0 mm
- added copper zone on B.Cu, net GND
Other:
- board size 16.5 x 19.8 mm -> 16.5 x 32.5 mm
Changed lines of the file:
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@@
 		)
 	)
+	(footprint "Capacitor_SMD:C_0603_1608Metric"
+		(layer "F.Cu")
+		(at 83.225 53.5 180)
+		(descr "Capacitor SMD 0603 (1608 Metric), square (rectangular) end terminal, IPC-7351 nominal, (Body size source: IPC-SM-782 page 76, https://www.pcb-3d.com/wordpress/wp-content/uploads/ipc-sm-782a_amendment_1_and_2.pdf)")
+		(tags "capacitor")
+		(property "Reference" "C2"
+			(at 0 -1.43 0)
+			(layer "F.SilkS")
+			(effects
+				(font
+					(size 1 1)
+					(thickness 0.15)
+				)
+			)
+		)
+		(property "Value" ".1UF"
+			(at 0 1.43 0)
+			(layer "F.Fab")
+			(effects
+				(font
+					(size 1 1)
+					(thickness 0.15)
+				)
+			)
+		)
+		(property "Datasheet" ""
+			(at 0 0 0)
+			(layer "F.Fab")
+			(hide yes)
+			(effects
+				(font
+					(size 1.27 1.27)
+				)
+			)
+		)
+		(property "Description" "Unpolarized capacitor"
+			(at 0 0 0)
+			(layer "F.Fab")
+			(hide yes)
+			(effects
+				(font
+					(size 1.27 1.27)
+				)
+			)
+		)
+		(property "KiLib_Generator" "SMD_2terminal_chip_molded"
+			(at 0 0 0)
+			(layer "F.SilkS")
+			(hide yes)
+			(effects
+				(font
+					(size 1 1)
+					(thickness 0.15)
+				)
+			)
+		)
+		(property ki_fp_filters "C_*")
+		(sheetname "/")
+		(sheetfile "light_blink.kicad_sch")
+		(units
+			(unit
+				(name "A")
+				(pins "1" "2")
+			)
+		)
+		(attr smd)
+		(duplicate_pad_numbers_are_jumpers no)
+		(fp_line
+			(start -0.14058 0.51)
+			(end 0.14058 0.51)
+			(stroke
+				(width 0.12)
+				(type solid)
+			)
+			(layer "F.SilkS")
+		)
+		(fp_line
+			(start -0.14058 -0.51)
+			(end 0.14058 -0.51)
+			(stroke
+				(width 0.12)
+				(type solid)
+			)
+			(layer "F.SilkS")
+		)
+		(fp_rect
+			(start -1.48 -0.73)
+			(end 1.48 0.73)
+			(stroke
+				(width 0.05)
+				(type solid)
+			)
+			(fill no)
+			(layer "F.CrtYd")
+		)
+		(fp_rect
+			(start -0.8 -0.4)
+			(end 0.8 0.4)
+			(stroke
+				(width 0.1)
+				(type solid)
+			)
+			(fill no)
+			(layer "F.Fab")
+		)
+		(fp_text user "${REFERENCE}"
+			(at 0 0 0)
+			(layer "F.Fab")
+			(effects
+				(font
+					(size 0.4 0.4)
+					(thickness 0.06)
+				)
+			)
+		)
+		(pad "1" smd roundrect
+			(at -0.775 0 180)
+			(size 0.9 0.95)
+			(layers "F.Cu" "F.Mask" "F.Paste")
+			(roundrect_rratio 0.25)
+			(net "Net-(U1-VOUT)")
+			(pintype "passive")
+		)
+		(pad "2" smd roundrect
+			(at 0.775 0 180)
+			(size 0.9 0.95)
+			(layers "F.Cu" "F.Mask" "F.Paste")
+			(roundrect_rratio 0.25)
+			(net "GND")
+			(pintype "passive")
+		)
+		(embedded_fonts no)
+		(model "${KICAD10_3DMODEL_DIR}/Capacitor_SMD.3dshapes/C_0603_1608Metric.step"
+			(offset
+				(xyz 0 0 0)
+			)
+			(scale
+				(xyz 1 1 1)
+			)
+			(rotate
+				(xyz 0 0 0)
+			)
+		)
+	)
 	(footprint "Resistor_SMD:R_0603_1608Metric"
 		(layer "F.Cu")
@@
 	(footprint "Resistor_SMD:R_0603_1608Metric"
 		(layer "F.Cu")
-		(at 83.82 58.483 -90)
+		(at 83.5 60.253 -90)
 		(descr "Resistor SMD 0603 (1608 Metric), square (rectangular) end terminal, IPC-7351 nominal, (Body size source: IPC-SM-782 page 72, https://www.pcb-3d.com/wordpress/wp-content/uploads/ipc-sm-782a_amendment_1_and_2.pdf)")
 		(tags "resistor")
@@
 	(footprint "Resistor_SMD:R_0603_1608Metric"
 		(layer "F.Cu")
-		(at 83.82 55.055 -90)
+		(at 83.5 56.825 -90)
 		(descr "Resistor SMD 0603 (1608 Metric), square (rectangular) end terminal, IPC-7351 nominal, (Body size source: IPC-SM-782 page 72, https://www.pcb-3d.com/wordpress/wp-content/uploads/ipc-sm-782a_amendment_1_and_2.pdf)")
 		(tags "resistor")
@@
 	)
 	(gr_rect
-		(start 69.85 45)
+		(start 69.85 32.258)
 		(end 86.36 64.77)
 		(stroke
@@
 	)
 	(segment
+		(start 82.5 55)
+		(end 81.638002 55)
+		(width 0.2)
+		(layer "F.Cu")
+		(net "Net-(U1-VOUT)")
+	)
+	(segment
+		(start 84 53.5)
+		(end 82.5 55)
+		(width 0.2)
+		(layer "F.Cu")
+		(net "Net-(U1-VOUT)")
+	)
+	(segment
 		(start 73.554001 56.134)
 		(end 74.422 56.134)
@@
 	)
 	(segment
-		(start 82.574602 55.649998)
-		(end 83.82 54.4046)
+		(start 82.924604 56)
+		(end 83.5 56)
 		(width 0.2)
 		(layer "F.Cu")
@@
 	)
 	(segment
-		(start 83.82 54.4046)
-		(end 83.82 54.23)
+		(start 81.638002 55.649998)
+		(end 82.574602 55.649998)
+		(width 0.2)
+		(layer "F.Cu")
+		(net "Net-(U3-VOUTB)")
+	)
+	(segment
+		(start 82.574602 55.649998)
+		(end 82.924604 56)
 		(width 0.2)
 		(layer "F.Cu")
@@
 	)
 	(segment
-		(start 81.638002 55.649998)
-		(end 82.574602 55.649998)
-		(width 0.2)
-		(layer "F.Cu")
-		(net "Net-(U3-VOUTB)")
-	)
-	(segment
 		(start 76.65 62.5)
 		(end 78.5 60.65)
@@
 	)
 	(segment
+		(start 82.45 53.5)
+		(end 81.5 53.5)
+		(width 0.2)
+		(layer "F.Cu")
+		(net "GND")
+	)
+	(segment
 		(start 73 59)
 		(end 75.050002 56.949998)
@@
 	)
 	(via
+		(at 81.5 53.5)
+		(size 0.6)
+		(drill 0.3)
+		(layers "F.Cu" "B.Cu")
+		(net "GND")
+	)
+	(via
 		(at 75.5 58)
 		(size 0.6096)
@@
 	)
 	(segment
+		(start 78 57)
+		(end 76 57)
+		(width 0.2)
+		(layer "B.Cu")
+		(net "GND")
+	)
+	(segment
 		(start 75.5 60)
 		(end 78 62.5)
@@
 	)
 	(segment
+		(start 81.5 53.5)
+		(end 78 57)
+		(width 0.2)
+		(layer "B.Cu")
+		(net "GND")
+	)
+	(segment
 		(start 83.82 62.358)
 		(end 83.946 62.484)
@@
 	)
 	(segment
-		(start 83.82 59.308)
+		(start 83.5 61.078)
+		(end 83.82 61.398)
+		(width 0.2)
+		(layer "F.Cu")
+		(net "Net-(R7-Pad1)")
+	)
+	(segment
+		(start 83.82 61.398)
 		(end 83.82 62.358)
 		(width 0.2)
@@
 	)
 	(segment
-		(start 83.82 55.88)
-		(end 83.82 57.658)
+		(start 83.5 57.65)
+		(end 83.5 59.428)
 		(width 0.2)
 		(layer "F.Cu")
 		(net "Net-(R8-Pad1)")
 	)
+	(zone
+		(net "GND")
+		(layer "B.Cu")
+		(hatch edge 0.5)
+		(connect_pads
+			(clearance 0.5)
+		)
+		(min_thickness 0.25)
+		(fill
+			(thermal_gap 0.5)
+			(thermal_bridge_width 0.5)
+			(island_removal_mode 0)
+		)
+		(polygon
+			(pts
+				(xy 70 32.5) (xy 86 32.5) (xy 86 64.5) (xy 70 64.5)
+			)
+		)
+	)
 	(embedded_fonts no)

Commit message: Add files via upload
Parts:
- added C3: .1UF, Capacitor_SMD:C_0603_1608Metric, F.Cu at (83.3, 53.5)
- added C4: 1UF, Capacitor_SMD:C_0603_1608Metric, F.Cu at (72.2, 57.0)
- added C5: 1UF, Capacitor_SMD:C_0603_1608Metric, F.Cu at (76.2, 53.0)
- C2: value .1UF -> 1UF
- moved J1 2.34 mm to (74.5, 49.5)
- moved U1 1.89 mm to (72.5, 53.8)
- moved C2 1.50 mm to (83.3, 52.0)
- moved R6 0.56 mm to (72.3, 59.5)
Routing:
- net GND: track 21.0 -> 37.1 mm, vias 3 -> 4
- net Net-(U1-VOUT): track 22.8 -> 26.8 mm
- net Net-(U1-VIN): track 3.30 -> 7.05 mm
- net Net-(R1-Pad1): track 7.54 -> 5.60 mm
- net Net-(U1-GND): track 11.4 -> 12.8 mm

Commit message: Add files via upload
Parts:
- removed U3: MCP6022T-I/ST, footprints:TSSOP8_MC_MCH
- added U2: MCP6021T-E/OT, footprints:SOT-23-5_MC_MCH, F.Cu at (78.3, 55.9)
- moved C3 2.28 mm to (81.0, 53.5)
- moved R9 2.03 mm to (81.5, 56.5)
- moved C2 1.78 mm to (81.5, 52.0)
- moved J1 0.71 mm to (74.0, 50.0)
Connections:
- J1 pad 4: Net-(U1-GND) -> GND
- U1 pad 1: Net-(U1-GND) -> GND
Routing:
- net Net-(U1-GND): track 12.8 -> 0.00 mm
- net GND: track 37.1 -> 41.6 mm, vias 4 -> 5
- net Net-(U1-VOUT): track 26.8 -> 25.1 mm
- net Net-(U2-VIN+): track 8.82 -> 10.4 mm
- net Net-(U2-VIN-): track 8.69 -> 7.11 mm
- net Net-(R8-Pad1): track 1.78 -> 2.93 mm
- net Net-(U2-VOUT): track 10.0 -> 11.2 mm
Other:
- board size 16.5 x 32.5 mm -> 16.5 x 22.3 mm
