File: light_blink.kicad_sch (KiCad schematic)
At the start: 14 parts, among them J1 CONN PLUG USB2.0 TYPEA 4POS R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, U1 MCP1702T-3302E/CB, U3 MCP6022T-I/ST

Commit message: Add files via upload
Parts:
- added C2: .1UF, Capacitor_SMD:C_0603_1608Metric, symbol Device:C
Connections:
- net GND: now also C2.2
- net at R5.2, U1.2 (VOUT), U3.8 (VDD): now also C2.1
Changed lines of the file:
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@@
+	)
+	(junction
+		(at 118.11 63.5)
+		(diameter 0)
+		(color 0 0 0 0)
 	)
 	(junction
@@
 	(wire
 		(pts
+			(xy 118.11 63.5) (xy 124.46 63.5)
+		)
+		(stroke
+			(width 0)
+			(type default)
+		)
+	)
+	(wire
+		(pts
 			(xy 134.62 110.49) (xy 134.62 116.84)
 		)
@@
 	(wire
 		(pts
-			(xy 115.57 63.5) (xy 124.46 63.5)
+			(xy 115.57 63.5) (xy 118.11 63.5)
 		)
 		(stroke
@@
 	)
 	(symbol
+		(lib_id "Device:C")
+		(at 118.11 67.31 0)
+		(unit 1)
+		(body_style 1)
+		(exclude_from_sim no)
+		(in_bom yes)
+		(on_board yes)
+		(in_pos_files yes)
+		(dnp no)
+		(fields_autoplaced yes)
+		(property "Reference" "C2"
+			(at 121.92 66.0399 0)
+			(show_name no)
+			(do_not_autoplace no)
+			(effects
+				(font
+					(size 1.27 1.27)
+				)
+				(justify left)
+			)
+		)
+		(property "Value" ".1UF"
+			(at 121.92 68.5799 0)
+			(show_name no)
+			(do_not_autoplace no)
+			(effects
+				(font
+					(size 1.27 1.27)
+				)
+				(justify left)
+			)
+		)
+		(property "Footprint" "Capacitor_SMD:C_0603_1608Metric"
+			(at 119.0752 71.12 0)
+			(hide yes)
+			(show_name no)
+			(do_not_autoplace no)
+			(effects
+				(font
+					(size 1.27 1.27)
+				)
+			)
+		)
+		(property "Datasheet" ""
+			(at 118.11 67.31 0)
+			(hide yes)
+			(show_name no)
+			(do_not_autoplace no)
+			(effects
+				(font
+					(size 1.27 1.27)
+				)
+			)
+		)
+		(property "Description" "Unpolarized capacitor"
+			(at 118.11 67.31 0)
+			(hide yes)
+			(show_name no)
+			(do_not_autoplace no)
+			(effects
+				(font
+					(size 1.27 1.27)
+				)
+			)
+		)
+		(pin "1"
+		)
+		(pin "2"
+		)
+		(instances
+			(project "light_blink"
+				(path "/4ddc1785-0852-42e4-b306-3ee70128813c"
+					(reference "C2")
+					(unit 1)
+				)
+			)
+		)
+	)
+	(symbol
 		(lib_id "Device:R")
 		(at 179.07 87.63 270)
@@
 					(unit 1)
 				)
+			)
+		)
+	)
+	(symbol
+		(lib_id "power:GND")
+		(at 118.11 71.12 0)
+		(unit 1)
+		(body_style 1)
+		(exclude_from_sim no)
+		(in_bom yes)
+		(on_board yes)
+		(in_pos_files yes)
+		(dnp no)
+		(fields_autoplaced yes)
+		(property "Reference" "#PWR06"
+			(at 118.11 77.47 0)
+			(hide yes)
+			(show_name no)
+			(do_not_autoplace no)
+			(effects
+				(font
+					(size 1.27 1.27)
+				)
+			)
+		)
+		(property "Value" "GND"
+			(at 118.11 76.2 0)
+			(show_name no)
+			(do_not_autoplace no)
+			(effects
+				(font
+					(size 1.27 1.27)
+				)
+			)
+		)
+		(property "Footprint" ""
+			(at 118.11 71.12 0)
+			(hide yes)
+			(show_name no)
+			(do_not_autoplace no)
+			(effects
+				(font
+					(size 1.27 1.27)
+				)
+			)
+		)
+		(property "Datasheet" ""
+			(at 118.11 71.12 0)
+			(hide yes)
+			(show_name no)
+			(do_not_autoplace no)
+			(effects
+				(font
+					(size 1.27 1.27)
+				)
+			)
+		)
+		(property "Description" "Power symbol creates a global label with name \"GND\" , ground"
+			(at 118.11 71.12 0)
+			(hide yes)
+			(show_name no)
+			(do_not_autoplace no)
+			(effects
+				(font
+					(size 1.27 1.27)
+				)
+			)
+		)
+		(pin "1"
+		)
+		(instances
+			(project "light_blink"
+				(path "/4ddc1785-0852-42e4-b306-3ee70128813c"
+					(reference "#PWR06")
+					(unit 1)
+				)

Commit message: Add files via upload
Parts:
- added C3: .1UF, Capacitor_SMD:C_0603_1608Metric, symbol Device:C
- added C4, C5: 1UF, Capacitor_SMD:C_0603_1608Metric, symbol Device:C
- C2: value .1UF -> 1UF
Connections:
- net GND: now also C3.2, C4.2, C5.2
- net at C2.1, R5.2, U1.2 (VOUT)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: now also C3.1, C4.1
- net at J1.1, U1.3 (VIN): now also C5.1

Commit message: Add files via upload
Parts:
- removed U3: MCP6022T-I/ST, footprints:TSSOP8_MC_MCH, symbol light_library:MCP6022T-I_ST
- added U2: MCP6021T-E/OT, footprints:SOT-23-5_MC_MCH, symbol light_library:MCP6021T-E_OT
Connections:
- net GND: now also J1.4, U1.1 (GND), U2.2 (VSS)
- net at R1.2, R2.2: now also U2.3 (VIN+)
- net at R2.1, R4.2, R9.1: now also U2.1 (VOUT)
- net at C2.1, C3.1, C4.1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: now also U2.5 (VDD)
- net at C1.1, R3.2: now also U2.4 (VIN-)
- no-connect marks 0 -> 2
